File: AVB Ethernet switch with Can bus/AVB switch with Can gateway.sch (KiCad schematic (older format))
At the start: 49 parts, among them J1 Molex_micro_fit_2X2, J2 Molex_micro_fit_2X2, J3 Molex_micro_fit_2X2, J4 RJ45_Magjack_Connector, J6 RJ45_Magjack_Connector, J7 RJ45_Magjack_Connector, J8 RJ45_Magjack_Connector, U1 LINEAR_LDO, U10 LINEAR_LDO, U11 LINEAR_LDO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

Commit message: change libery
Parts:
- C1, C10, C11, C12, C13, C14, C15, C2, C3, C5, C6, C68, C69, C7, C70, C71, C72, C73, C75, C76, C77, C78, C8, C9: footprint Capacitors_SMD:C_0603_HandSoldering -> Capacitor_SMD:C_0603_1608Metric_Pad1.05x0.95mm_HandSolder
- J1, J2, J3: footprint AVB switch with Can gateway:Molex micro_fir 2X2 -> AVB switch with Can gateway:Molex_micro_fit_2X2; symbol AVB-switch-with-Can-gateway-rescue:Molex_micro_fit_2X2-Rj45 -> AVB-switch-with-Can-gateway-rescue:Molex_micro_fit_2X2-Rj45-AVB-switch-with-Can-gateway-rescue
- J4, J6, J7, J8: symbol AVB-switch-with-Can-gateway-rescue:RJ45_Magjack_Connector-Rj45 -> AVB-switch-with-Can-gateway-rescue:RJ45_Magjack_Connector-Rj45-AVB-switch-with-Can-gateway-rescue
- R14, R15, R16, R17, R18, R19, R20, R21: footprint Resistors_SMD:R_0603_HandSoldering -> Resistor_SMD:R_0603_1608Metric_Pad1.05x0.95mm_HandSolder
- U1, U10, U11, U12, U2, U3: footprint TO_SOT_Packages_SMD:SOT-223 -> Package_TO_SOT_SMD:SOT-223; symbol AVB-switch-with-can:LINEAR_LDO -> AVB-switch-with-Can-gateway-rescue:LINEAR_LDO-AVB-switch-with-can
