File: AVB Ethernet switch with Can bus/mcu_stm32_1.sch (KiCad schematic (older format))
At the start: 34 parts, among them J10 Conn_01x02, J5 Conn_01x04, J9 Conn_02x04_Counter_Clockwise, U4 STM32F765VITx, U5 SN65HVD234, U6 SN65HVD234, U7 SN65HVD234, Y2 Crystal-8Mhz

Commit message: change libery
Parts:
- C16, C17, C18, C19, C20, C21, C22, C23, C24, C25, C26, C27, C28: footprint Capacitors_SMD:C_0603_HandSoldering -> Capacitor_SMD:C_0603_1608Metric_Pad1.05x0.95mm_HandSolder; symbol AVB-switch-with-Can-gateway-rescue:CC0603KRX7R7BB104-symbols-Can-Gateway-rescue -> AVB-switch-with-Can-gateway-rescue:CC0603KRX7R7BB104-symbols-Can-Gateway-rescue-AVB-switch-with-Can-gateway-rescue
- C79, C80, FB2: footprint Capacitors_SMD:C_0603_HandSoldering -> Capacitor_SMD:C_0603_1608Metric_Pad1.05x0.95mm_HandSolder
- J10: footprint Pin_Headers:Pin_Header_Straight_1x02_Pitch2.54mm -> Connector_PinHeader_2.54mm:PinHeader_1x02_P2.54mm_Vertical
- J5: footprint Pin_Headers:Pin_Header_Straight_1x04_Pitch2.54mm -> Connector_PinHeader_2.54mm:PinHeader_1x04_P2.54mm_Vertical
- J9: footprint Pin_Headers:Pin_Header_Straight_2x04_Pitch2.54mm -> Connector_PinHeader_2.54mm:PinHeader_2x04_P2.54mm_Vertical
- R1: footprint Capacitors_SMD:C_0603_HandSoldering -> Resistor_SMD:R_0603_1608Metric_Pad1.05x0.95mm_HandSolder
- R10, R11, R12, R4, R5, R6, R7, R8, R9: footprint Resistors_SMD:R_0603_HandSoldering -> Resistor_SMD:R_0603_1608Metric_Pad1.05x0.95mm_HandSolder
- U4: footprint Housings_QFP:LQFP-100_14x14mm_Pitch0.5mm -> Package_QFP:LQFP-100_14x14mm_P0.5mm
- U5, U6, U7: footprint Housings_SOIC:SOIC-8_3.9x4.9mm_Pitch1.27mm -> Package_SO:SOIC-8_3.9x4.9mm_P1.27mm
- Y2: footprint Crystals:Crystal_SMD_3225-4pin_3.2x2.5mm -> Crystal:Crystal_SMD_3225-4Pin_3.2x2.5mm
