File: AVB Ethernet switch with Can bus/switch.sch (KiCad schematic (older format))
At the start: 68 parts, among them IC1 KSZ8567STXI-TR, J11 Conn_01x02, J12 Conn_01x02, J13 Conn_01x02, J14 Conn_01x02, J15 Conn_01x02, J16 Conn_01x02, Y1 Crystal-25Mhz

Commit message: change libery
Parts:
- C29, C30, C31, C32, C33, C34, C35, C36, C37, C38, C39, C4, C40, C41, C42, C43, C44, C45, C46, C47, C48, C49, C50, C51, C52, C53, C54, C55, C56, C57, C58, C59, C60, C61, C62, C63, C64, C65, C66, C67, C74, FB3, FB4, FB5, FB6: footprint Capacitors_SMD:C_0603_HandSoldering -> Capacitor_SMD:C_0603_1608Metric_Pad1.05x0.95mm_HandSolder
- D4, D5: footprint Diodes_SMD:D_SOD-323_HandSoldering -> Diode_SMD:D_SOD-323_HandSoldering
- IC1: symbol AVB-switch-with-Can-gateway-rescue:KSZ8567STXI-TR-KSZ8567STXI-TR -> AVB-switch-with-Can-gateway-rescue:KSZ8567STXI-TR-KSZ8567STXI-TR-AVB-switch-with-Can-gateway-rescue
- J11, J12, J13, J14, J15, J16: footprint Pin_Headers:Pin_Header_Straight_1x02_Pitch2.54mm -> Connector_PinHeader_2.54mm:PinHeader_1x02_P2.54mm_Vertical
- R13, R2, R22, R23, R24, R25, R26, R27, R28, R29, R3, R30, R31: footprint Resistors_SMD:R_0603_HandSoldering -> Resistor_SMD:R_0603_1608Metric_Pad1.05x0.95mm_HandSolder
- Y1: footprint Crystals:Crystal_SMD_3225-4pin_3.2x2.5mm -> Crystal:Crystal_SMD_3225-4Pin_3.2x2.5mm
