File: AVB_Ethernet_switch_with_CAN_bus/AVB switch with Can gateway.kicad_pcb (KiCad board)
At the start: 4 copper layers, 137 x 55 mm, 151 parts, among them IC1 KSZ8567STXI-TR, J1 Molex_micro_fit_2X2, J10 Conn_01x02, J11 Conn_01x02, J12 Conn_01x02, J13 Conn_01x02, J14 Conn_01x02, J15 Conn_01x02, J16 Conn_01x02, J2 Molex_micro_fit_2X2, J3 Molex_micro_fit_2X2, J4 RJ45_Magjack_Connector, J5 Conn_01x04, J6 RJ45_Magjack_Connector, J7 RJ45_Magjack_Connector, J8 RJ45_Magjack_Connector, J9 Conn_02x04_Counter_Clockwise, U1 LINEAR_LDO, U10 LINEAR_LDO, U11 LINEAR_LDO, U12 LINEAR_LDO, U2 LINEAR_LDO, U3 LINEAR_LDO, U4 STM32F765VITx, U5 SN65HVD234, U6 SN65HVD234, U7 SN65HVD234, Y1 Crystal-25Mhz, Y2 Crystal-8Mhz

Commit message: set README file
Parts:
- C1, C10, C11, C12, C13, C14, C15, C16, C17, C18, C19, C2, C20, C21, C22, C23, C24, C25, C26, C27, C28, C29, C3, C30, C31, C32, C33, C34, C35, C36, C37, C38, C39, C4, C40, C41, C42, C43, C44, C45, C46, C47, C48, C49, C5, C50, C51, C52, C53, C54, C55, C56, C57, C58, C59, C6, C60, C61, C62, C63, C64, C65, C66, C67, C68, C69, C7, C70, C71, C72, C73, C74, C75, C76, C77, C78, C79, C8, C80, C9, FB2, FB3, FB4, FB5, FB6: footprint Capacitors_SMD:C_0603_HandSoldering -> Capacitor_SMD:C_0603_1608Metric_Pad1.05x0.95mm_HandSolder
- D4, D5: footprint Diodes_SMD:D_SOD-323_HandSoldering -> Diode_SMD:D_SOD-323_HandSoldering
- J1, J2, J3: footprint AVB switch with Can gateway:Molex micro_fir 2X2 -> AVB switch with Can gateway:Molex_micro_fit_2X2
- J10, J11, J12, J13, J14, J15, J16: footprint Pin_Headers:Pin_Header_Straight_1x02_Pitch2.54mm -> Connector_PinHeader_2.54mm:PinHeader_1x02_P2.54mm_Vertical
- J5: footprint Pin_Headers:Pin_Header_Straight_1x04_Pitch2.54mm -> Connector_PinHeader_2.54mm:PinHeader_1x04_P2.54mm_Vertical
- J9: footprint Pin_Headers:Pin_Header_Straight_2x04_Pitch2.54mm -> Connector_PinHeader_2.54mm:PinHeader_2x04_P2.54mm_Vertical
- R1: footprint Capacitors_SMD:C_0603_HandSoldering -> Resistor_SMD:R_0603_1608Metric_Pad1.05x0.95mm_HandSolder
- R10, R11, R12, R13, R14, R15, R16, R17, R18, R19, R2, R20, R21, R22, R23, R24, R25, R26, R27, R28, R29, R3, R30, R31, R4, R5, R6, R7, R8, R9: footprint Resistors_SMD:R_0603_HandSoldering -> Resistor_SMD:R_0603_1608Metric_Pad1.05x0.95mm_HandSolder
- U1, U10, U11, U12, U2, U3: footprint TO_SOT_Packages_SMD:SOT-223 -> Package_TO_SOT_SMD:SOT-223
- U4: footprint Housings_QFP:LQFP-100_14x14mm_Pitch0.5mm -> Package_QFP:LQFP-100_14x14mm_P0.5mm
- U5, U6, U7: footprint Housings_SOIC:SOIC-8_3.9x4.9mm_Pitch1.27mm -> Package_SO:SOIC-8_3.9x4.9mm_P1.27mm
- Y1, Y2: footprint Crystals:Crystal_SMD_3225-4pin_3.2x2.5mm -> Crystal:Crystal_SMD_3225-4Pin_3.2x2.5mm
